File: ares-parachute-board.kicad_sch (KiCad schematic)
At the start: 53 parts, among them J1 Conn_01x16_Female, J2 Conn_01x16_Female, J3 Conn_01x02_Male, J4 Conn_ARM_JTAG_SWD_10, J5 Conn_01x03_Pin, J6 MPT 0.5/2-2.54, U1 XC6206P332MR, U2 AP2552W6-7, U3 SR05-ES, U4 W25Q128JVSIQTR, U5 LIS2DW12TR, U6 STM32F103CBTx, U7 LIS2DW12TR, X1 CSTNE8M00G520000R0, X2 Q13FC1350000400

Commit message: layout done
Parts:
- removed J2: Conn_01x16_Female, Connector_PinHeader_2.54mm:PinHeader_1x16_P2.54mm_Vertical, symbol Connector:Conn_01x16_Female
Connections:
- net +3.3V: now also J1.2 (Pin_2); no longer J1.1 (Pin_1)
- net +5V: now also J1.1 (Pin_1), JP1.3 (B); no longer J1.3 (Pin_3), JP1.1 (A)
- net GND: now also J1.3 (Pin_3); no longer J1.2 (Pin_2)
- net PA3: no longer J1.16 (Pin_16)
- net PB0: now also J1.9 (Pin_9); no longer J1.6 (Pin_6)
- net PB1: now also J1.10 (Pin_10); no longer J1.7 (Pin_7)
- net PB12: now also J1.15 (Pin_15); no longer J1.12 (Pin_12)
- net PB13: now also J1.14 (Pin_14); no longer J1.13 (Pin_13)
- net PB14: now also J1.13 (Pin_13); no longer J1.14 (Pin_14)
- net PB15: now also J1.12 (Pin_12); no longer J1.15 (Pin_15)
- net PB2: now also J1.11 (Pin_11); no longer J1.8 (Pin_8)
- net PB5: now also J1.6 (Pin_6); no longer J1.9 (Pin_9)
- net PB8: now also J1.7 (Pin_7); no longer J1.10 (Pin_10)
- net PB9: now also J1.8 (Pin_8); no longer J1.11 (Pin_11)
- net at R15.2: now also JP1.1 (A); no longer JP1.3 (B)
- no-connect marks 27 -> 14

Commit message: added testpoints, not on board yet
Parts:
- added T1, T2, T3, T4, T5, T6, T7: RH-5000, easyeda_exported:TEST-TH_BD2.54-P1.4_RED, symbol easyeda_exported:RH-5000
Connections:
- net I2C1_SCL: now also T1.1
- net I2C1_SDA: now also T2.1
- net I2C2_SCL: now also T3.1
- net I2C2_SDA: now also T4.1
- net SPI1_MISO: now also T5.1
- net SPI1_MOSI: now also T6.1
- net SPI1_SCK: now also T7.1
- no-connect marks 14 -> 15
Other:
- note added: "Prototype Test Points"
- moved on the sheet: LED2, LED3, LED4, R12, R13, R14
