File: ares-parachute-board.kicad_sch (KiCad schematic)
At the start: 59 parts, among them J1 Conn_01x16_Female, J3 Conn_01x02_Male, J4 Conn_ARM_JTAG_SWD_10, J5 Conn_01x03_Pin, J6 MPT 0.5/2-2.54, T1 RH-5000, T2 RH-5000, T3 RH-5000, T4 RH-5000, T5 RH-5000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

Commit message: update board for prototype 2
Parts:
- removed C10, C8: 12.5p, Capacitor_SMD:C_0603_1608Metric, symbol Device:C
- removed R9: 0, Resistor_SMD:R_0603_1608Metric, symbol Device:R
- removed T1, T2, T3, T4, T5, T6, T7: RH-5000, easyeda_exported:TEST-TH_BD2.54-P1.4_RED, symbol easyeda_exported:RH-5000
- removed X2: Q13FC1350000400, easyeda_exported:FC-135R_L3.2-W1.5, symbol easyeda_exported:Q13FC1350000400
- added SW1: TS-1187A-B-A-B, easyeda_exported:SW-SMD_4P-L5.1-W5.1-P3.70-LS6.5-TL_H1.5, symbol easyeda_exported:TS-1187A-B-A-B
- added U8: DSIC-02-TS-GER, easyeda_exported:SW-SMD_DSIC-02-TS-GER, symbol easyeda_exported:DSIC-02-TS-GER
- R12, R13: value 270 -> 560
- R14: value 100 -> 2k2
- R5, R6: value 5.1k -> 5k1
Connections:
- net GND: now also SW1.1 (A), SW1.3 (C)
- net I2C1_SCL: now also U8.4; no longer R7.2, U5.1 (SCL/SPC)
- net I2C2_SCL: now also U8.3; no longer R10.2, U7.1 (SCL/SPC)
- net ~{MEM_CS}: now also U6.29 (PA8)
- net ~{RESET}: now also SW1.2 (B), SW1.4 (D)
- net at X1.3: now also U6.6 (PD1)
- new net I2C1_SCL_DC: R7.2, U5.1 (SCL/SPC), U8.1
- new net I2C2_SCL_DC: R10.2, U7.1 (SCL/SPC), U8.2
Other:
- note added: "DIP switch to disconnect I2Cs to simulate error case"
- note added: "Pin for SPI_CS?"
- note added: "To do: - Pin 1 ident debug"
- note removed: "32.768kHz Crystal"
- note removed: "Prototype Test Points"
- moved on the sheet: X1

Commit message: ordered version 1.0
Parts:
- C1, C6: LCSC (none) -> C1671
- C11, C12, C13, C14, C16, C5, C7, C9: LCSC (none) -> C14663
- C15: LCSC (none) -> C19666
- C2, C3: LCSC (none) -> C15849
- C4: LCSC (none) -> C19702
- J4: LCSC (none) -> C7501289
- LED1, LED2: LCSC (none) -> C84256
- LED3: LCSC (none) -> C2296
- LED4: LCSC (none) -> C2297
- R1, R2: LCSC (none) -> C23140
- R10, R11, R7, R8: LCSC (none) -> C23162
- R12, R13: LCSC (none) -> C23204
- R14: LCSC (none) -> C4190
- R15: LCSC (none) -> C22775
- R3: LCSC (none) -> C22966
- R4: LCSC (none) -> C23206
- R5, R6: LCSC (none) -> C23186
- SW1: LCSC (none) -> C318884
- U1: LCSC (none) -> C5446
- U2: LCSC (none) -> C441824
- U3: LCSC (none) -> C5180250
- U4: LCSC (none) -> C97521
- U5, U7: LCSC (none) -> C189624
- U6: LCSC (none) -> C8304
- U8: LCSC (none) -> C7471373
- USB1: LCSC (none) -> C393939
- X1: LCSC (none) -> C907975

Commit message: fix error in reset button placement for future revision
Connections:
- net GND: now also SW1.4 (D); no longer SW1.1 (A)
- net ~{RESET}: now also SW1.1 (A); no longer SW1.4 (D)
Other:
- note removed: "5mA each: Red, Yellow Vf 2.0V -> 260 Ohm ~ 270 Ohm Green Vf 2.8V -> 100 Ohm"
- note removed: "Pin for SPI_CS?"
- note removed: "To do: - Pin 1 ident debug"
- moved on the sheet: SW1
Changed lines of the file:
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@@
 	(title_block
 		(title "ARES Parachute Board")
-		(date "2025-01-21")
-		(rev "PROTO2")
+		(date "2025-02-14")
+		(rev "v1.1")
 		(company "Hochschule Luzern, Technik & Architektur")
 		(comment 1 "Peter Allenspach")
 	)
 	(junction
-		(at 231.14 133.35)
-		(diameter 0)
-		(color 0 0 0 0)
-	)
-	(junction
 		(at 140.97 40.64)
 		(diameter 0)
@@
 	)
 	(junction
+		(at 231.14 137.16)
+		(diameter 0)
+		(color 0 0 0 0)
+	)
+	(junction
 		(at 74.93 106.68)
 		(diameter 0)
@@
 	)
 	(junction
-		(at 231.14 123.19)
-		(diameter 0)
-		(color 0 0 0 0)
-	)
-	(junction
 		(at 231.14 77.47)
 		(diameter 0)
@@
 	(wire
 		(pts
+			(xy 226.06 132.08) (xy 226.06 137.16)
+		)
+		(stroke
+			(width 0)
+			(type default)
+		)
+	)
+	(wire
+		(pts
 			(xy 135.89 111.76) (xy 146.05 111.76)
 		)
@@
 	(wire
 		(pts
+			(xy 236.22 132.08) (xy 236.22 137.16)
+		)
+		(stroke
+			(width 0)
+			(type default)
+		)
+	)
+	(wire
+		(pts
 			(xy 180.34 143.51) (xy 180.34 147.32)
 		)
@@
 	(wire
 		(pts
+			(xy 226.06 120.65) (xy 236.22 120.65)
+		)
+		(stroke
+			(width 0)
+			(type default)
+		)
+	)
+	(wire
+		(pts
 			(xy 71.12 146.05) (xy 73.66 146.05)
 		)
@@
 	(wire
 		(pts
-			(xy 229.87 77.47) (xy 231.14 77.47)
+			(xy 226.06 137.16) (xy 231.14 137.16)
 		)
 		(stroke
@@
 	(wire
 		(pts
-			(xy 31.75 90.17) (xy 31.75 88.9)
+			(xy 229.87 77.47) (xy 231.14 77.47)
 		)
 		(stroke
@@
 	(wire
 		(pts
-			(xy 247.65 142.24) (xy 260.35 142.24)
+			(xy 31.75 90.17) (xy 31.75 88.9)
 		)
 		(stroke
@@
 	(wire
 		(pts
-			(xy 41.91 175.26) (xy 41.91 170.18)
+			(xy 247.65 142.24) (xy 260.35 142.24)
 		)
 		(stroke
@@
 	(wire
 		(pts
-			(xy 190.5 135.89) (xy 196.85 135.89)
+			(xy 41.91 175.26) (xy 41.91 170.18)
 		)
 		(stroke
@@
 	(wire
 		(pts
-			(xy 224.79 36.83) (xy 224.79 43.18)
+			(xy 190.5 135.89) (xy 196.85 135.89)
 		)
 		(stroke
@@
 	(wire
 		(pts
-			(xy 40.64 31.75) (xy 43.18 31.75)
+			(xy 224.79 36.83) (xy 224.79 43.18)
 		)
 		(stroke
@@
 	(wire
 		(pts
-			(xy 186.69 45.72) (xy 203.2 45.72)
+			(xy 40.64 31.75) (xy 43.18 31.75)
 		)
 		(stroke
@@
 	(wire
 		(pts
-			(xy 231.14 123.19) (xy 237.49 123.19)
+			(xy 186.69 45.72) (xy 203.2 45.72)
 		)
 		(stroke
@@
 	(wire
 		(pts
+			(xy 226.06 124.46) (xy 226.06 120.65)
+		)
+		(stroke
+			(width 0)
+			(type default)
+		)
+	)
+	(wire
+		(pts
 			(xy 234.95 36.83) (xy 241.3 36.83)
 		)
@@
 	(wire
 		(pts
-			(xy 231.14 120.65) (xy 231.14 123.19)
-		)
-		(stroke
-			(width 0)
-			(type default)
-		)
-	)
-	(wire
-		(pts
 			(xy 40.64 39.37) (xy 43.18 39.37)
 		)
@@
 	(wire
 		(pts
-			(xy 231.14 133.35) (xy 237.49 133.35)
-		)
-		(stroke
-			(width 0)
-			(type default)
-		)
-	)
-	(wire
-		(pts
 			(xy 251.46 62.23) (xy 251.46 64.77)
 		)
@@
 	(wire
 		(pts
-			(xy 229.87 133.35) (xy 231.14 133.35)
-		)
-		(stroke
-			(width 0)
-			(type default)
-		)
-	)
-	(wire
-		(pts
 			(xy 186.69 40.64) (xy 191.77 40.64)
 		)
@@
 	(wire
 		(pts
+			(xy 236.22 137.16) (xy 231.14 137.16)
+		)
+		(stroke
+			(width 0)
+			(type default)
+		)
+	)
+	(wire
+		(pts
 			(xy 40.64 49.53) (xy 43.18 49.53)
 		)
@@
 	(wire
 		(pts
-			(xy 40.64 29.21) (xy 43.18 29.21)
+			(xy 236.22 124.46) (xy 236.22 120.65)
 		)
 		(stroke
@@
 	(wire
 		(pts
-			(xy 30.48 134.62) (xy 39.37 134.62)
+			(xy 40.64 29.21) (xy 43.18 29.21)
 		)
 		(stroke
@@
 	(wire
 		(pts
-			(xy 40.64 105.41) (xy 17.78 105.41)
+			(xy 30.48 134.62) (xy 39.37 134.62)
 		)
 		(stroke
@@
 	(wire
 		(pts
-			(xy 41.91 170.18) (xy 49.53 170.18)
+			(xy 40.64 105.41) (xy 17.78 105.41)
 		)
 		(stroke
@@
 	(wire
 		(pts
-			(xy 179.07 88.9) (xy 181.61 88.9)
+			(xy 41.91 170.18) (xy 49.53 170.18)
 		)
 		(stroke
@@
 	(wire
 		(pts
-			(xy 135.89 142.24) (xy 146.05 142.24)
+			(xy 179.07 88.9) (xy 181.61 88.9)
 		)
 		(stroke
@@
 	(wire
 		(pts
-			(xy 135.89 139.7) (xy 146.05 139.7)
+			(xy 135.89 142.24) (xy 146.05 142.24)
 		)
 		(stroke
@@
 	(wire
 		(pts
-			(xy 242.57 21.59) (xy 242.57 22.86)
+			(xy 135.89 139.7) (xy 146.05 139.7)
 		)
 		(stroke
@@
 	(wire
 		(pts
-			(xy 231.14 133.35) (xy 231.14 137.16)
+			(xy 242.57 21.59) (xy 242.57 22.86)
 		)
 		(stroke
@@
 	(wire
 		(pts
-			(xy 229.87 123.19) (xy 231.14 123.19)
-		)
-		(stroke
-			(width 0)
-			(type default)
-		)
-	)
-	(wire
-		(pts
 			(xy 53.34 186.69) (xy 41.91 186.69)
 		)
@@
 		)
 	)
-	(text "To do:\n- Pin 1 ident debug"
-		(exclude_from_sim no)
-		(at 212.598 114.3 0)
-		(effects
-			(font
-				(size 1.27 1.27)
-			)
-		)
-	)
 	(text "PA2"
 		(exclude_from_sim no)
@@
 		)
 	)
-	(text "Pin for SPI_CS?"
-		(exclude_from_sim no)
-		(at 209.55 96.52 0)
-		(effects
-			(font
-				(size 1.27 1.27)
-			)
-		)
-	)
 	(text "NOR Flash"
 		(exclude_from_sim no)
@@
 		)
 	)
-	(text "5mA each:\nRed, Yellow Vf 2.0V -> 260 Ohm ~ 270 Ohm\nGreen Vf 2.8V -> 100 Ohm"
-		(exclude_from_sim no)
-		(at 157.48 194.818 0)
-		(effects
-			(font
-				(size 0.762 0.762)
-			)
-		)
-	)
 	(text "Vf ~ 2V"
 		(exclude_from_sim no)
@@
 	(symbol
 		(lib_id "easyeda_exported:TS-1187A-B-A-B")
-		(at 232.41 128.27 90)
+		(at 231.14 127 0)
 		(unit 1)
 		(exclude_from_sim no)
@@
 		(on_board yes)
 		(dnp no)
-		(fields_autoplaced yes)
 		(property "Reference" "SW1"
-			(at 238.76 126.9999 90)
+			(at 235.204 125.984 0)
 			(effects
 				(font
 					(size 1.27 1.27)
 				)
-				(justify right)
 			)
 		)
 		(property "Value" "TS-1187A-B-A-B"
-			(at 238.76 129.5399 90)
+			(at 241.554 128.524 0)
 			(effects
 				(font
 					(size 1.27 1.27)
 				)
-				(justify right)
 			)
 		)
 		(property "Footprint" "easyeda_exported:SW-SMD_4P-L5.1-W5.1-P3.70-LS6.5-TL_H1.5"
-			(at 245.11 128.27 0)
+			(at 231.14 139.7 0)
 			(effects
 				(font
@@
 		)
 		(property "Datasheet" "https://lcsc.com/product-detail/Tactile-Switches_XKB-Enterprise-TS-1187-B-A-A_C318884.html"
-			(at 247.65 128.27 0)
+			(at 231.14 142.24 0)
 			(effects
 				(font
@@
 		)
 		(property "Description" ""
-			(at 232.41 128.27 0)
+			(at 231.14 127 0)
 			(effects
 				(font
@@
 		)
 		(property "LCSC Part" "C318884"
-			(at 250.19 128.27 0)
+			(at 231.14 144.78 0)
 			(effects
 				(font
@@
 		)
 		(property "LCSC" "C318884"
-			(at 238.76 126.9999 0)
+			(at 232.4101 133.35 0)
 			(effects
 				(font
